File: FEAR-16 - Shield - CathReg.kicad_pcb (KiCad board)
At the start: 4 copper layers, 60.3 x 39.2 mm, 63 parts, among them J101 Supply, J102 Signals, J103 Channel-In, Q201 NDFPD1N150CG, U201 OPA2156xD, U202 OPA2156xD, U203 OPA2156xD, U204 OPA2156xD

Commit message: V1.3 (improved fine-tuning of CF- and UD-Amps)
PCB Changes:
 - Amplification Poti (1Meg) changed to Offset-Resistor (100k) + Poti (50k) to achieve 20x finer tuning of the amplification

Misc.:
 - Fixed .gitignore to ignore the prl files
Parts:
- added R212: 100k, Resistor_SMD:R_0603_1608Metric, B.Cu at (30.4, 5.69)
- added R213: 100k, Resistor_SMD:R_0603_1608Metric, B.Cu at (50.0, 19.8)
- C222, C223: value 68n/25V -> 220n/25V
- R205, R210: value 50R -> 100k
- RV201, RV202: value 1M -> 50k
Connections:
- C222 pad 2: Net-(R209-Pad2) -> Net-(U204B--)
- C223 pad 2: Net-(R204-Pad2) -> Net-(U202B--)
- R204 pad 2: Net-(R204-Pad2) -> Net-(U202B--)
- R209 pad 2: Net-(R209-Pad2) -> Net-(U204B--)
- RV201 pad 1: Net-(R204-Pad2) -> Net-(R212-Pad2)
- RV201 pad 2: Net-(R204-Pad2) -> Net-(R212-Pad2)
- RV202 pad 1: Net-(R209-Pad2) -> Net-(R213-Pad2)
- RV202 pad 2: Net-(R209-Pad2) -> Net-(R213-Pad2)
- U202 pad 6: Net-(R204-Pad2) -> Net-(U202B--)
- U204 pad 6: Net-(R209-Pad2) -> Net-(U204B--)
Routing:
- net Net-(R209-Pad2): track 18.6 -> 0.00 mm, vias 1 -> 0
- net Net-(R204-Pad2): track 17.1 -> 0.00 mm, vias 1 -> 0
- net Net-(U204B--): track 0.00 -> 9.78 mm, vias 0 -> 1
- net Net-(U202B--): track 0.00 -> 9.38 mm, vias 0 -> 1
- net Net-(R212-Pad2): track 0.00 -> 5.16 mm
- net Net-(R213-Pad2): track 0.00 -> 5.16 mm
Other:
- board text added: "V1.3"
- board text removed: "V1.2"
